Commit message: Add my_robot_description

File: my_robot_description/urdf/my_robot.urdf.xacro (robot description, xacro)
@@ -1,4 +1,5 @@
 <?xml version="1.0"?>
 <robot xmlns:xacro="http://ros.org/wiki/xacro" name="my_robot">
+  <!-- xacro properties -->
   <xacro:property name="platform_length" value="0.5"/>
   <xacro:property name="platform_width" value="0.5"/>
@@ -9,6 +10,25 @@
   <xacro:property name="track_length" value="0.5"/>
   <xacro:property name="track_width" value="0.1"/>
-  <xacro:property name="track_height" value="0.15"/>
+  <xacro:property name="track_height" value="0.1"/>
+  <!-- LiDAR properties: diameter 5cm (radius 2.5cm), height 3cm -->
+  <xacro:property name="lidar_radius" value="0.025"/>
+  <xacro:property name="lidar_height" value="0.03"/>
+  <!-- World link: the root of the robot model, used to avoid KDL parser warning -->
+  <link name="world"/>
+  <!-- Connect world link to base_link (since base_link is now the first substantial link) -->
+  <joint name="world_to_base_link" type="fixed">
+    <parent link="world"/>
+    <child link="base_link"/>
+    <origin xyz="0 0 0" rpy="0 0 0"/>
+  </joint>
   <link name="base_link">
+    <!-- Base link needs an inertial block for Gazebo simulation -->
+    <inertial>
+      <mass value="0.001"/>
+      <origin xyz="0 0 0" rpy="0 0 0"/>
+      <inertia ixx="0.000001" ixy="0.0" ixz="0.0"
+               iyy="0.000001" iyz="0.0"
+               izz="0.000001"/>
+    </inertial>
   </link>
   <link name="bottom_plate">
@@ -22,4 +42,12 @@
       </material>
     </visual>
+    <!-- Inertial block for bottom_plate -->
+    <inertial>
+      <mass value="0.5"/>
+      <origin xyz="0 0 0" rpy="0 0 0"/>
+      <inertia ixx="0.01" ixy="0.0" ixz="0.0"
+               iyy="0.01" iyz="0.0"
+               izz="0.01"/>
+    </inertial>
   </link>
   <joint name="base_to_bottom" type="fixed">
@@ -36,4 +64,12 @@
       <material name="yellow"/>
     </visual>
+    <!-- Inertial block for main_body -->
+    <inertial>
+      <mass value="1.0"/>
+      <origin xyz="0 0 0" rpy="0 0 0"/>
+      <inertia ixx="0.05" ixy="0.0" ixz="0.0"
+               iyy="0.05" iyz="0.0"
+               izz="0.05"/>
+    </inertial>
   </link>
   <joint name="bottom_to_body" type="fixed">
@@ -50,4 +86,12 @@
       <material name="yellow"/>
     </visual>
+    <!-- Inertial block for top_plate -->
+    <inertial>
+      <mass value="0.5"/>
+      <origin xyz="0 0 0" rpy="0 0 0"/>
+      <inertia ixx="0.01" ixy="0.0" ixz="0.0"
+               iyy="0.01" iyz="0.0"
+               izz="0.01"/>
+    </inertial>
   </link>
   <joint name="body_to_top" type="fixed">
@@ -66,4 +110,12 @@
       </material>
     </visual>
+    <!-- Inertial block for left_track -->
+    <inertial>
+      <mass value="0.2"/>
+      <origin xyz="0 0 0" rpy="0 0 0"/>
+      <inertia ixx="0.005" ixy="0.0" ixz="0.0"
+               iyy="0.005" iyz="0.0"
+               izz="0.005"/>
+    </inertial>
   </link>
   <joint name="base_to_left_track" type="fixed">
@@ -80,4 +132,12 @@
       <material name="black"/>
     </visual>
+    <!-- Inertial block for right_track -->
+    <inertial>
+      <mass value="0.2"/>
+      <origin xyz="0 0 0" rpy="0 0 0"/>
+      <inertia ixx="0.005" ixy="0.0" ixz="0.0"
+               iyy="0.005" iyz="0.0"
+               izz="0.005"/>
+    </inertial>
   </link>
   <joint name="base_to_right_track" type="fixed">
@@ -86,3 +146,66 @@
     <origin xyz="0 ${-(platform_width/2 + 0.01 - track_width/2)} ${-platform_thickness/2 - track_height/2}" rpy="0 0 0"/>
   </joint>
+  <!-- LiDAR Sensor Link -->
+  <link name="lidar_link">
+    <visual>
+      <geometry>
+        <cylinder radius="${lidar_radius}" length="${lidar_height}"/>
+      </geometry>
+      <origin xyz="0 0 0" rpy="0 0 0"/>
+      <material name="Red">
+        <color rgba="1 0 0 1"/>
+      </material>
+    </visual>
+    <!-- Inertial block for lidar_link -->
+    <inertial>
+      <mass value="0.05"/>
+      <origin xyz="0 0 0" rpy="0 0 0"/>
+      <inertia ixx="0.0001" ixy="0.0" ixz="0.0"
+               iyy="0.0001" iyz="0.0"
+               izz="0.0001"/>
+    </inertial>
+  </link>
+  <!-- Joint to attach LiDAR to top_plate -->
+  <joint name="lidar_joint" type="fixed">
+    <parent link="top_plate"/>
+    <child link="lidar_link"/>
+    <!-- Position LiDAR on top of the top_plate -->
+    <origin xyz="0 0 ${platform_thickness/2 + lidar_height/2}" rpy="0 0 0"/>
+  </joint>
+  <!-- Gazebo-specific extensions (now part of the main xacro file) -->
+  <gazebo reference="lidar_link">
+    <sensor name="lidar" type="gpu_lidar">
+      <pose>0 0 0 0 0 0</pose>
+      <topic>/scan</topic>
+      <update_rate>10</update_rate>
+      <ray>
+        <scan>
+          <horizontal>
+            <samples>640</samples>
+            <resolution>1</resolution>
+            <min_angle>-3.14</min_angle>
+            <max_angle>3.14</max_angle>
+          </horizontal>
+          <vertical>
+            <samples>1</samples>
+            <resolution>0.01</resolution>
+            <min_angle>0</min_angle>
+            <max_angle>0</max_angle>
+          </vertical>
+        </scan>
+        <range>
+          <min>0.1</min>
+          <max>10.0</max>
+          <resolution>0.01</resolution>
+        </range>
+      </ray>
+      <always_on>1</always_on>
+      <visualize>true</visualize>
+    </sensor>
+  </gazebo>
+  <gazebo>
+    <plugin filename="gz-sim-sensors-system" name="gz::sim::systems::Sensors">
+      <render_engine>ogre2</render_engine>
+    </plugin>
+  </gazebo>
 </robot>

Commit message: Assignment 4

File: my_robot_description/urdf/my_robot.urdf.xacro (robot description, xacro)
@@ -16,5 +16,5 @@
   <!-- World link: the root of the robot model, used to avoid KDL parser warning -->
   <link name="world"/>
-  <!-- Connect world link to base_link (since base_link is now the first substantial link) -->
+  <!-- Connect world link to base_link -->
   <joint name="world_to_base_link" type="fixed">
     <parent link="world"/>
@@ -24,4 +24,19 @@
   <link name="base_link">
     <!-- Base link needs an inertial block for Gazebo simulation -->
+    <visual>
+      <geometry>
+        <box size="0.001 0.001 0.001"/>
+      </geometry>
+      <origin xyz="0 0 0" rpy="0 0 0"/>
+      <material name="Green">
+        <color rgba="0 1 0 1"/>
+      </material>
+    </visual>
+    <collision>
+      <geometry>
+        <box size="0.001 0.001 0.001"/>
+      </geometry>
+      <origin xyz="0 0 0" rpy="0 0 0"/>
+    </collision>
     <inertial>
       <mass value="0.001"/>
@@ -42,5 +57,10 @@
       </material>
     </visual>
-    <!-- Inertial block for bottom_plate -->
+    <collision>
+      <geometry>
+        <box size="${platform_length} ${platform_width} ${platform_thickness}"/>
+      </geometry>
+      <origin xyz="0 0 0" rpy="0 0 0"/>
+    </collision>
     <inertial>
       <mass value="0.5"/>
@@ -64,5 +84,10 @@
       <material name="yellow"/>
     </visual>
-    <!-- Inertial block for main_body -->
+    <collision>
+      <geometry>
+        <box size="${body_length} ${body_width} ${body_height}"/>
+      </geometry>
+      <origin xyz="0 0 0" rpy="0 0 0"/>
+    </collision>
     <inertial>
       <mass value="1.0"/>
@@ -86,5 +111,10 @@
       <material name="yellow"/>
     </visual>
-    <!-- Inertial block for top_plate -->
+    <collision>
+      <geometry>
+        <box size="${platform_length} ${platform_width} ${platform_thickness}"/>
+      </geometry>
+      <origin xyz="0 0 0" rpy="0 0 0"/>
+    </collision>
     <inertial>
       <mass value="0.5"/>
@@ -110,5 +140,10 @@
       </material>
     </visual>
-    <!-- Inertial block for left_track -->
+    <collision>
+      <geometry>
+        <box size="${track_length} ${track_width} ${track_height}"/>
+      </geometry>
+      <origin xyz="0 0 0" rpy="0 0 0"/>
+    </collision>
     <inertial>
       <mass value="0.2"/>
@@ -132,5 +167,10 @@
       <material name="black"/>
     </visual>
-    <!-- Inertial block for right_track -->
+    <collision>
+      <geometry>
+        <box size="${track_length} ${track_width} ${track_height}"/>
+      </geometry>
+      <origin xyz="0 0 0" rpy="0 0 0"/>
+    </collision>
     <inertial>
       <mass value="0.2"/>
@@ -157,5 +197,10 @@
       </material>
     </visual>
-    <!-- Inertial block for lidar_link -->
+    <collision>
+      <geometry>
+        <cylinder radius="${lidar_radius}" length="${lidar_height}"/>
+      </geometry>
+      <origin xyz="0 0 0" rpy="0 0 0"/>
+    </collision>
     <inertial>
       <mass value="0.05"/>
@@ -173,5 +218,5 @@
     <origin xyz="0 0 ${platform_thickness/2 + lidar_height/2}" rpy="0 0 0"/>
   </joint>
-  <!-- Gazebo-specific extensions (now part of the main xacro file) -->
+  <!-- Gazebo-specific extensions (sensors and plugins) -->
   <gazebo reference="lidar_link">
     <sensor name="lidar" type="gpu_lidar">
