Commit message: New model

File: my_robot_description/urdf/my_robot.urdf.xacro (robot description, xacro)
@@ -1,256 +1,162 @@
 <?xml version="1.0"?>
-<robot xmlns:xacro="http://ros.org/wiki/xacro" name="my_robot">
-  <!-- xacro properties -->
-  <xacro:property name="platform_length" value="0.5"/>
-  <xacro:property name="platform_width" value="0.5"/>
-  <xacro:property name="platform_thickness" value="0.01"/>
-  <xacro:property name="body_length" value="0.5"/>
+<robot xmlns:xacro="http://www.ros.org/wiki/xacro" name="my_robot">
+  <!-- ======================= คุณสมบัติต่างๆ (Properties) ======================= -->
+  <xacro:property name="body_length" value="0.35"/>
   <xacro:property name="body_width" value="0.3"/>
-  <xacro:property name="body_height" value="0.1"/>
+  <xacro:property name="body_height" value="0.2"/>
   <xacro:property name="track_length" value="0.5"/>
   <xacro:property name="track_width" value="0.1"/>
-  <xacro:property name="track_height" value="0.1"/>
-  <!-- LiDAR properties: diameter 5cm (radius 2.5cm), height 3cm -->
+  <xacro:property name="track_height" value="0.18"/>
   <xacro:property name="lidar_radius" value="0.025"/>
   <xacro:property name="lidar_height" value="0.03"/>
-  <!-- World link: the root of the robot model, used to avoid KDL parser warning -->
-  <link name="world"/>
-  <!-- Connect world link to base_link -->
-  <joint name="world_to_base_link" type="fixed">
-    <parent link="world"/>
-    <child link="base_link"/>
-    <origin xyz="0 0 0" rpy="0 0 0"/>
-  </joint>
+  <xacro:property name="wheel_radius" value="0.025"/>
+  <xacro:property name="wheel_thickness" value="0.001"/>
+  <xacro:property name="wheel_z_offset" value="-0.07"/>
+  <xacro:property name="top_plate_length" value="0.5"/>
+  <xacro:property name="top_plate_width" value="0.5"/>
+  <xacro:property name="top_plate_thickness" value="0.003"/>
+  <xacro:property name="lidar_stand_length" value="0.5"/>
+  <xacro:property name="lidar_stand_width" value="0.3"/>
+  <xacro:property name="lidar_stand_height" value="0.1"/>
+  <!-- ## NEW: คุณสมบัติสำหรับ Plate วาง Lidar ## -->
+  <xacro:property name="lidar_plate_length" value="0.5"/>
+  <xacro:property name="lidar_plate_width" value="0.5"/>
+  <xacro:property name="lidar_plate_thickness" value="0.003"/>
+  <!-- ======================= สีของวัสดุ (Materials) ======================= -->
+  <material name="black"><color rgba="0.1 0.1 0.1 1.0"/></material>
+  <material name="yellow"><color rgba="1.0 1.0 0.0 1.0"/></material>
+  <material name="red"><color rgba="1 0 0 1"/></material>
+  <material name="white"><color rgba="1.0 1.0 1.0 1.0"/></material>
+  <!-- ======================= โครงสร้างหุ่นยนต์ (Robot Structure) ======================= -->
+  <link name="base_footprint"/>
   <link name="base_link">
-    <!-- Base link needs an inertial block for Gazebo simulation -->
     <visual>
-      <geometry>
-        <box size="0.001 0.001 0.001"/>
-      </geometry>
-      <origin xyz="0 0 0" rpy="0 0 0"/>
-      <material name="Green">
-        <color rgba="0 1 0 1"/>
-      </material>
+      <geometry><box size="${body_length} ${body_width} ${body_height}"/></geometry>
+      <material name="yellow"/>
     </visual>
     <collision>
-      <geometry>
-        <box size="0.001 0.001 0.001"/>
-      </geometry>
-      <origin xyz="0 0 0" rpy="0 0 0"/>
+      <geometry><box size="${body_length*0.9} ${body_width*0.9} ${body_height*0.9}"/></geometry>
     </collision>
     <inertial>
-      <mass value="0.001"/>
-      <origin xyz="0 0 0" rpy="0 0 0"/>
-      <inertia ixx="0.000001" ixy="0.0" ixz="0.0"
-               iyy="0.000001" iyz="0.0"
-               izz="0.000001"/>
+      <mass value="5.0"/>
+      <inertia ixx="0.4" ixy="0" ixz="0" iyy="0.4" iyz="0" izz="0.2"/>
     </inertial>
   </link>
-  <link name="bottom_plate">
+  <joint name="base_footprint_joint" type="fixed">
+    <parent link="base_footprint"/>
+    <child link="base_link"/>
+    <origin xyz="0 0 ${wheel_radius - wheel_z_offset}"/>
+  </joint>
+  <xacro:macro name="track_housing" params="prefix side">
+    <link name="${prefix}_track">
+      <visual>
+        <geometry><box size="${track_length} ${track_width} ${track_height}"/></geometry>
+        <material name="black"/>
+      </visual>
+    </link>
+    <joint name="base_to_${prefix}_track" type="fixed">
+      <parent link="base_link"/>
+      <child link="${prefix}_track"/>
+      <origin xyz="0 ${side * (body_width/2 + track_width/2)} ${-body_height/2 + track_height/2}"/>
+    </joint>
+  </xacro:macro>
+  <xacro:track_housing prefix="left" side="1"/>
+  <xacro:track_housing prefix="right" side="-1"/>
+  <xacro:macro name="drive_wheel" params="prefix side">
+    <link name="${prefix}_wheel">
+      <visual>
+        <origin rpy="${pi/2} 0 0"/>
+        <geometry><cylinder radius="${wheel_radius}" length="${wheel_thickness}"/></geometry>
+        <material name="white"/>
+      </visual>
+      <collision>
+        <origin rpy="${pi/2} 0 0"/>
+        <geometry><cylinder radius="${wheel_radius}" length="${wheel_thickness}"/></geometry>
+      </collision>
+      <inertial>
+        <mass value="0.5"/>
+        <inertia ixx="0.001" ixy="0" ixz="0" iyy="0.001" iyz="0" izz="0.001"/>
+      </inertial>
+    </link>
+    <joint name="${prefix}_wheel_joint" type="continuous">
+      <parent link="base_link"/>
+      <child link="${prefix}_wheel"/>
+      <origin xyz="0 ${side * (body_width/2 + track_width + wheel_thickness/2)} ${wheel_z_offset}"/>
+      <axis xyz="0 1 0"/>
+    </joint>
+  </xacro:macro>
+  <xacro:drive_wheel prefix="left"  side="1"/>
+  <xacro:drive_wheel prefix="right" side="-1"/>
+  <link name="top_plate">
     <visual>
-      <geometry>
-        <box size="${platform_length} ${platform_width} ${platform_thickness}"/>
-      </geometry>
-      <origin xyz="0 0 0" rpy="0 0 0"/>
-      <material name="yellow">
-        <color rgba="1.0 1.0 0.0 1.0"/>
-      </material>
+      <geometry><box size="${top_plate_length} ${top_plate_width} ${top_plate_thickness}"/></geometry>
+      <material name="yellow"/>
     </visual>
     <collision>
-      <geometry>
-        <box size="${platform_length} ${platform_width} ${platform_thickness}"/>
-      </geometry>
-      <origin xyz="0 0 0" rpy="0 0 0"/>
+      <geometry><box size="${top_plate_length} ${top_plate_width} ${top_plate_thickness}"/></geometry>
     </collision>
     <inertial>
       <mass value="0.5"/>
-      <origin xyz="0 0 0" rpy="0 0 0"/>
-      <inertia ixx="0.01" ixy="0.0" ixz="0.0"
-               iyy="0.01" iyz="0.0"
-               izz="0.01"/>
+      <inertia ixx="0.01" ixy="0" ixz="0" iyy="0.01" iyz="0" izz="0.01"/>
     </inertial>
   </link>
-  <joint name="base_to_bottom" type="fixed">
+  <joint name="top_plate_joint" type="fixed">
     <parent link="base_link"/>
-    <child link="bottom_plate"/>
-    <origin xyz="0 0 0" rpy="0 0 0"/>
+    <child link="top_plate"/>
+    <origin xyz="0 0 ${body_height/2 + top_plate_thickness/2}"/>
   </joint>
-  <link name="main_body">
+  <link name="lidar_stand">
     <visual>
-      <geometry>
-        <box size="${body_length} ${body_width} ${body_height}"/>
-      </geometry>
-      <origin xyz="0 0 0" rpy="0 0 0"/>
+      <geometry><box size="${lidar_stand_length} ${lidar_stand_width} ${lidar_stand_height}"/></geometry>
       <material name="yellow"/>
     </visual>
     <collision>
-      <geometry>
-        <box size="${body_length} ${body_width} ${body_height}"/>
-      </geometry>
-      <origin xyz="0 0 0" rpy="0 0 0"/>
+      <geometry><box size="${lidar_stand_length} ${lidar_stand_width} ${lidar_stand_height}"/></geometry>
     </collision>
     <inertial>
-      <mass value="1.0"/>
-      <origin xyz="0 0 0" rpy="0 0 0"/>
-      <inertia ixx="0.05" ixy="0.0" ixz="0.0"
-               iyy="0.05" iyz="0.0"
-               izz="0.05"/>
+      <mass value="0.2"/>
+      <inertia ixx="0.01" ixy="0" ixz="0" iyy="0.01" iyz="0" izz="0.01"/>
     </inertial>
   </link>
-  <joint name="bottom_to_body" type="fixed">
-    <parent link="bottom_plate"/>
-    <child link="main_body"/>
-    <origin xyz="0 0 ${platform_thickness/2 + body_height/2}" rpy="0 0 0"/>
+  <joint name="lidar_stand_joint" type="fixed">
+    <parent link="top_plate"/>
+    <child link="lidar_stand"/>
+    <origin xyz="0 0 ${top_plate_thickness/2 + lidar_stand_height/2}"/>
   </joint>
-  <link name="top_plate">
+  <!-- ## NEW: สร้าง Plate สำหรับวาง Lidar ## -->
+  <link name="lidar_plate">
     <visual>
-      <geometry>
-        <box size="${platform_length} ${platform_width} ${platform_thickness}"/>
-      </geometry>
-      <origin xyz="0 0 0" rpy="0 0 0"/>
+      <geometry><box size="${lidar_plate_length} ${lidar_plate_width} ${lidar_plate_thickness}"/></geometry>
       <material name="yellow"/>
     </visual>
     <collision>
-      <geometry>
-        <box size="${platform_length} ${platform_width} ${platform_thickness}"/>
-      </geometry>
-      <origin xyz="0 0 0" rpy="0 0 0"/>
+      <geometry><box size="${lidar_plate_length} ${lidar_plate_width} ${lidar_plate_thickness}"/></geometry>
     </collision>
     <inertial>
-      <mass value="0.5"/>
-      <origin xyz="0 0 0" rpy="0 0 0"/>
-      <inertia ixx="0.01" ixy="0.0" ixz="0.0"
-               iyy="0.01" iyz="0.0"
-               izz="0.01"/>
+      <mass value="0.1"/>
+      <inertia ixx="1e-6" ixy="0" ixz="0" iyy="1e-6" iyz="0" izz="1e-6"/>
     </inertial>
   </link>
-  <joint name="body_to_top" type="fixed">
-    <parent link="main_body"/>
-    <child link="top_plate"/>
-    <origin xyz="0 0 ${body_height/2 + platform_thickness/2}" rpy="0 0 0"/>
+  <joint name="lidar_plate_joint" type="fixed">
+    <parent link="lidar_stand"/>
+    <child link="lidar_plate"/>
+    <origin xyz="0 0 ${lidar_stand_height/2 + lidar_plate_thickness/2}"/>
   </joint>
-  <link name="left_track">
+  <link name="lidar_link">
     <visual>
-      <geometry>
-        <box size="${track_length} ${track_width} ${track_height}"/>
-      </geometry>
-      <origin xyz="0 0 0" rpy="0 0 0"/>
-      <material name="black">
-        <color rgba="0.1 0.1 0.1 1.0"/>
-      </material>
+      <geometry><cylinder radius="${lidar_radius}" length="${lidar_height}"/></geometry>
+      <material name="red"/>
     </visual>
     <collision>
-      <geometry>
-        <box size="${track_length} ${track_width} ${track_height}"/>
-      </geometry>
-      <origin xyz="0 0 0" rpy="0 0 0"/>
+      <geometry><cylinder radius="${lidar_radius}" length="${lidar_height}"/></geometry>
     </collision>
-    <inertial>
-      <mass value="0.2"/>
-      <origin xyz="0 0 0" rpy="0 0 0"/>
-      <inertia ixx="0.005" ixy="0.0" ixz="0.0"
-               iyy="0.005" iyz="0.0"
-               izz="0.005"/>
-    </inertial>
+    <inertial><mass value="0.1"/><inertia ixx="1e-6" ixy="0" ixz="0" iyy="1e-6" iyz="0" izz="1e-6"/></inertial>
   </link>
-  <joint name="base_to_left_track" type="fixed">
-    <parent link="base_link"/>
-    <child link="left_track"/>
-    <origin xyz="0 ${platform_width/2 + 0.01 - track_width/2} ${-platform_thickness/2 - track_height/2}" rpy="0 0 0"/>
+  <joint name="lidar_joint" type="fixed">
+    <!-- ## FIX: ย้าย Lidar ไปยึดกับ Plate ที่สร้างขึ้นใหม่ ## -->
+    <parent link="lidar_plate"/>
+    <child link="lidar_link"/>
+    <origin xyz="0 0 ${lidar_plate_thickness/2 + lidar_height/2}"/>
   </joint>
-  <link name="right_track">
-    <visual>
-      <geometry>
-        <box size="${track_length} ${track_width} ${track_height}"/>
-      </geometry>
-      <origin xyz="0 0 0" rpy="0 0 0"/>
-      <material name="black"/>
-    </visual>
-    <collision>
-      <geometry>
-        <box size="${track_length} ${track_width} ${track_height}"/>
-      </geometry>
-      <origin xyz="0 0 0" rpy="0 0 0"/>
-    </collision>
-    <inertial>
-      <mass value="0.2"/>
-      <origin xyz="0 0 0" rpy="0 0 0"/>
-      <inertia ixx="0.005" ixy="0.0" ixz="0.0"
-               iyy="0.005" iyz="0.0"
-               izz="0.005"/>
-    </inertial>
-  </link>
-  <joint name="base_to_right_track" type="fixed">
-    <parent link="base_link"/>
-    <child link="right_track"/>
-    <origin xyz="0 ${-(platform_width/2 + 0.01 - track_width/2)} ${-platform_thickness/2 - track_height/2}" rpy="0 0 0"/>
-  </joint>
-  <!-- LiDAR Sensor Link -->
-  <link name="lidar_link">
-    <visual>
-      <geometry>
-        <cylinder radius="${lidar_radius}" length="${lidar_height}"/>
-      </geometry>
-      <origin xyz="0 0 0" rpy="0 0 0"/>
-      <material name="Red">
-        <color rgba="1 0 0 1"/>
-      </material>
-    </visual>
-    <collision>
-      <geometry>
-        <cylinder radius="${lidar_radius}" length="${lidar_height}"/>
-      </geometry>
-      <origin xyz="0 0 0" rpy="0 0 0"/>
-    </collision>
-    <inertial>
-      <mass value="0.05"/>
-      <origin xyz="0 0 0" rpy="0 0 0"/>
-      <inertia ixx="0.0001" ixy="0.0" ixz="0.0"
-               iyy="0.0001" iyz="0.0"
-               izz="0.0001"/>
-    </inertial>
-  </link>
-  <!-- Joint to attach LiDAR to top_plate -->
-  <joint name="lidar_joint" type="fixed">
-    <parent link="top_plate"/>
-    <child link="lidar_link"/>
-    <!-- Position LiDAR on top of the top_plate -->
-    <origin xyz="0 0 ${platform_thickness/2 + lidar_height/2}" rpy="0 0 0"/>
-  </joint>
-  <!-- Gazebo-specific extensions (sensors and plugins) -->
-  <gazebo reference="lidar_link">
-    <sensor name="lidar" type="gpu_lidar">
-      <pose>0 0 0 0 0 0</pose>
-      <topic>/scan</topic>
-      <update_rate>10</update_rate>
-      <ray>
-        <scan>
-          <horizontal>
-            <samples>640</samples>
-            <resolution>1</resolution>
-            <min_angle>-3.14</min_angle>
-            <max_angle>3.14</max_angle>
-          </horizontal>
-          <vertical>
-            <samples>1</samples>
-            <resolution>0.01</resolution>
-            <min_angle>0</min_angle>
-            <max_angle>0</max_angle>
-          </vertical>
-        </scan>
-        <range>
-          <min>0.1</min>
-          <max>10.0</max>
-          <resolution>0.01</resolution>
-        </range>
-      </ray>
-      <always_on>1</always_on>
-      <visualize>true</visualize>
-    </sensor>
-  </gazebo>
-  <gazebo>
-    <plugin filename="gz-sim-sensors-system" name="gz::sim::systems::Sensors">
-      <render_engine>ogre2</render_engine>
-    </plugin>
-  </gazebo>
+  <xacro:include filename="my_robot.gazebo.xacro" />
 </robot>

Commit message: Add Odom

File: my_robot_description/urdf/my_robot.urdf.xacro (robot description, xacro)
@@ -24,17 +24,29 @@
   <xacro:property name="lidar_plate_thickness" value="0.003"/>
   <!-- ======================= สีของวัสดุ (Materials) ======================= -->
-  <material name="black"><color rgba="0.1 0.1 0.1 1.0"/></material>
-  <material name="yellow"><color rgba="1.0 1.0 0.0 1.0"/></material>
-  <material name="red"><color rgba="1 0 0 1"/></material>
-  <material name="white"><color rgba="1.0 1.0 1.0 1.0"/></material>
+  <material name="black">
+    <color rgba="0.1 0.1 0.1 1.0"/>
+  </material>
+  <material name="yellow">
+    <color rgba="1.0 1.0 0.0 1.0"/>
+  </material>
+  <material name="red">
+    <color rgba="1 0 0 1"/>
+  </material>
+  <material name="white">
+    <color rgba="1.0 1.0 1.0 1.0"/>
+  </material>
   <!-- ======================= โครงสร้างหุ่นยนต์ (Robot Structure) ======================= -->
   <link name="base_footprint"/>
   <link name="base_link">
     <visual>
-      <geometry><box size="${body_length} ${body_width} ${body_height}"/></geometry>
+      <geometry>
+        <box size="${body_length} ${body_width} ${body_height}"/>
+      </geometry>
       <material name="yellow"/>
     </visual>
     <collision>
-      <geometry><box size="${body_length*0.9} ${body_width*0.9} ${body_height*0.9}"/></geometry>
+      <geometry>
+        <box size="${body_length*0.9} ${body_width*0.9} ${body_height*0.9}"/>
+      </geometry>
     </collision>
     <inertial>
@@ -51,5 +63,7 @@
     <link name="${prefix}_track">
       <visual>
-        <geometry><box size="${track_length} ${track_width} ${track_height}"/></geometry>
+        <geometry>
+          <box size="${track_length} ${track_width} ${track_height}"/>
+        </geometry>
         <material name="black"/>
       </visual>
@@ -67,10 +81,14 @@
       <visual>
         <origin rpy="${pi/2} 0 0"/>
-        <geometry><cylinder radius="${wheel_radius}" length="${wheel_thickness}"/></geometry>
+        <geometry>
+          <cylinder radius="${wheel_radius}" length="${wheel_thickness}"/>
+        </geometry>
         <material name="white"/>
       </visual>
       <collision>
         <origin rpy="${pi/2} 0 0"/>
-        <geometry><cylinder radius="${wheel_radius}" length="${wheel_thickness}"/></geometry>
+        <geometry>
+          <cylinder radius="${wheel_radius}" length="${wheel_thickness}"/>
+        </geometry>
       </collision>
       <inertial>
@@ -86,13 +104,17 @@
     </joint>
   </xacro:macro>
-  <xacro:drive_wheel prefix="left"  side="1"/>
+  <xacro:drive_wheel prefix="left" side="1"/>
   <xacro:drive_wheel prefix="right" side="-1"/>
   <link name="top_plate">
     <visual>
-      <geometry><box size="${top_plate_length} ${top_plate_width} ${top_plate_thickness}"/></geometry>
+      <geometry>
+        <box size="${top_plate_length} ${top_plate_width} ${top_plate_thickness}"/>
+      </geometry>
       <material name="yellow"/>
     </visual>
     <collision>
-      <geometry><box size="${top_plate_length} ${top_plate_width} ${top_plate_thickness}"/></geometry>
+      <geometry>
+        <box size="${top_plate_length} ${top_plate_width} ${top_plate_thickness}"/>
+      </geometry>
     </collision>
     <inertial>
@@ -108,9 +130,13 @@
   <link name="lidar_stand">
     <visual>
-      <geometry><box size="${lidar_stand_length} ${lidar_stand_width} ${lidar_stand_height}"/></geometry>
+      <geometry>
+        <box size="${lidar_stand_length} ${lidar_stand_width} ${lidar_stand_height}"/>
+      </geometry>
       <material name="yellow"/>
     </visual>
     <collision>
-      <geometry><box size="${lidar_stand_length} ${lidar_stand_width} ${lidar_stand_height}"/></geometry>
+      <geometry>
+        <box size="${lidar_stand_length} ${lidar_stand_width} ${lidar_stand_height}"/>
+      </geometry>
     </collision>
     <inertial>
@@ -127,9 +153,13 @@
   <link name="lidar_plate">
     <visual>
-      <geometry><box size="${lidar_plate_length} ${lidar_plate_width} ${lidar_plate_thickness}"/></geometry>
+      <geometry>
+        <box size="${lidar_plate_length} ${lidar_plate_width} ${lidar_plate_thickness}"/>
+      </geometry>
       <material name="yellow"/>
     </visual>
     <collision>
-      <geometry><box size="${lidar_plate_length} ${lidar_plate_width} ${lidar_plate_thickness}"/></geometry>
+      <geometry>
+        <box size="${lidar_plate_length} ${lidar_plate_width} ${lidar_plate_thickness}"/>
+      </geometry>
     </collision>
     <inertial>
@@ -145,11 +175,18 @@
   <link name="lidar_link">
     <visual>
-      <geometry><cylinder radius="${lidar_radius}" length="${lidar_height}"/></geometry>
+      <geometry>
+        <cylinder radius="${lidar_radius}" length="${lidar_height}"/>
+      </geometry>
       <material name="red"/>
     </visual>
     <collision>
-      <geometry><cylinder radius="${lidar_radius}" length="${lidar_height}"/></geometry>
+      <geometry>
+        <cylinder radius="${lidar_radius}" length="${lidar_height}"/>
+      </geometry>
     </collision>
-    <inertial><mass value="0.1"/><inertia ixx="1e-6" ixy="0" ixz="0" iyy="1e-6" iyz="0" izz="1e-6"/></inertial>
+    <inertial>
+      <mass value="0.1"/>
+      <inertia ixx="1e-6" ixy="0" ixz="0" iyy="1e-6" iyz="0" izz="1e-6"/>
+    </inertial>
   </link>
   <joint name="lidar_joint" type="fixed">
