Commit message: Nav2

File: my_robot_description/urdf/my_robot.gazebo.xacro (robot description, xacro)
@@ -3,7 +3,5 @@
   <!-- ======================= ปลั๊กอินทั่วไป (General Plugins) ======================= -->
   <gazebo>
-    <plugin
-      filename="gz-sim-sensors-system"
-      name="gz::sim::systems::Sensors">
+    <plugin filename="gz-sim-sensors-system" name="gz::sim::systems::Sensors">
     </plugin>
   </gazebo>
@@ -33,14 +31,10 @@
   <!-- ======================= ปลั๊กอินสำหรับสถานะข้อต่อ (Joint States) ======================= -->
   <gazebo>
-    <plugin
-      filename="gz-sim-joint-state-publisher-system"
-      name="gz::sim::systems::JointStatePublisher">
+    <plugin filename="gz-sim-joint-state-publisher-system" name="gz::sim::systems::JointStatePublisher">
     </plugin>
   </gazebo>
   <!-- ======================= ปลั๊กอินสำหรับขับเคลื่อน (Drive Plugin) ======================= -->
   <gazebo>
-    <plugin
-      filename="gz-sim-diff-drive-system"
-      name="gz::sim::systems::DiffDrive">
+    <plugin filename="gz-sim-diff-drive-system" name="gz::sim::systems::DiffDrive">
       <left_joint>left_wheel_joint</left_joint>
       <right_joint>right_wheel_joint</right_joint>
@@ -48,4 +42,7 @@
       <wheel_radius>${wheel_radius}</wheel_radius>
       <topic>cmd_vel</topic>
+      <publish_odom_tf>true</publish_odom_tf>
+      <frame_id>odom</frame_id>
+      <child_frame_id>base_footprint</child_frame_id>
     </plugin>
   </gazebo>

File: my_robot_description/urdf/my_robot.urdf.xacro (robot description, xacro)
@@ -10,5 +10,5 @@
   <xacro:property name="lidar_radius" value="0.025"/>
   <xacro:property name="lidar_height" value="0.03"/>
-  <xacro:property name="wheel_radius" value="0.025"/>
+  <xacro:property name="wheel_radius" value="0.021"/>
   <xacro:property name="wheel_thickness" value="0.001"/>
   <xacro:property name="wheel_z_offset" value="-0.07"/>

Commit message: Add mappinh

File: my_robot_description/urdf/my_robot.gazebo.xacro (robot description, xacro)
@@ -1,7 +1,9 @@
 <?xml version="1.0"?>
 <robot xmlns:xacro="http://www.ros.org/wiki/xacro">
+  <!-- Main sensor manager -->
   <gazebo>
     <plugin filename="gz-sim-sensors-system" name="gz::sim::systems::Sensors"/>
   </gazebo>
+  <!-- Lidar Sensor -->
   <gazebo reference="lidar_link">
     <sensor name="lidar_link" type="gpu_lidar">
@@ -23,6 +25,14 @@
         </range>
       </lidar>
-      </sensor>
+    </sensor>
   </gazebo>
+  <!-- IMU Sensor Plugin -->
+  <gazebo reference="imu_link">
+    <sensor name="imu_sensor" type="imu">
+      <topic>imu</topic>
+      <update_rate>50</update_rate>
+    </sensor>
+  </gazebo>
+  <!-- Joint State Publisher -->
   <gazebo>
     <plugin filename="gz-sim-joint-state-publisher-system" name="gz::sim::systems::JointStatePublisher">
@@ -30,4 +40,5 @@
     </plugin>
   </gazebo>
+  <!-- Differential Drive -->
   <gazebo>
     <plugin filename="gz-sim-diff-drive-system" name="gz::sim::systems::DiffDrive">

File: my_robot_description/urdf/my_robot.urdf.xacro (robot description, xacro)
@@ -1,5 +1,5 @@
 <?xml version="1.0"?>
 <robot xmlns:xacro="http://www.ros.org/wiki/xacro" name="my_robot">
-  <!-- ======================= คุณสมบัติต่างๆ (Properties) ======================= -->
+  <!-- ======================= Properties ======================= -->
   <xacro:property name="body_length" value="0.35"/>
   <xacro:property name="body_width" value="0.3"/>
@@ -19,9 +19,10 @@
   <xacro:property name="lidar_stand_width" value="0.3"/>
   <xacro:property name="lidar_stand_height" value="0.1"/>
-  <!-- ## NEW: คุณสมบัติสำหรับ Plate วาง Lidar ## -->
   <xacro:property name="lidar_plate_length" value="0.5"/>
   <xacro:property name="lidar_plate_width" value="0.5"/>
   <xacro:property name="lidar_plate_thickness" value="0.003"/>
-  <!-- ======================= สีของวัสดุ (Materials) ======================= -->
+  <!-- ## NEW: IMU Box Size ## -->
+  <xacro:property name="imu_size" value="0.02"/>
+  <!-- ======================= Materials ======================= -->
   <material name="black">
     <color rgba="0.1 0.1 0.1 1.0"/>
@@ -36,5 +37,5 @@
     <color rgba="1.0 1.0 1.0 1.0"/>
   </material>
-  <!-- ======================= โครงสร้างหุ่นยนต์ (Robot Structure) ======================= -->
+  <!-- ======================= Robot Structure ======================= -->
   <link name="base_footprint"/>
   <link name="base_link">
@@ -59,4 +60,27 @@
     <child link="base_link"/>
     <origin xyz="0 0 ${wheel_radius - wheel_z_offset}"/>
+  </joint>
+  <!-- ## NEW: IMU Sensor Link and Joint ## -->
+  <link name="imu_link">
+    <inertial>
+      <mass value="0.01"/>
+      <inertia ixx="1e-6" ixy="0" ixz="0" iyy="1e-6" iyz="0" izz="1e-6"/>
+    </inertial>
+    <visual>
+      <geometry>
+        <box size="${imu_size} ${imu_size} ${imu_size}"/>
+      </geometry>
+      <material name="red"/>
+    </visual>
+    <collision>
+      <geometry>
+        <box size="${imu_size} ${imu_size} ${imu_size}"/>
+      </geometry>
+    </collision>
+  </link>
+  <joint name="imu_joint" type="fixed">
+    <parent link="base_link"/>
+    <child link="imu_link"/>
+    <origin xyz="0 0 0"/>
   </joint>
   <xacro:macro name="track_housing" params="prefix side">
@@ -150,5 +174,4 @@
     <origin xyz="0 0 ${top_plate_thickness/2 + lidar_stand_height/2}"/>
   </joint>
-  <!-- ## NEW: สร้าง Plate สำหรับวาง Lidar ## -->
   <link name="lidar_plate">
     <visual>
@@ -191,5 +214,4 @@
   </link>
   <joint name="lidar_joint" type="fixed">
-    <!-- ## FIX: ย้าย Lidar ไปยึดกับ Plate ที่สร้างขึ้นใหม่ ## -->
     <parent link="lidar_plate"/>
     <child link="lidar_link"/>
